Commit message: fix: make joints revolute

File: urdf/r2d2-example.urdf (robot description, URDF)
Before this commit: robot visual, 16 links, 15 joints
Joints:
- joint gripper_extension: limit (none) -> lower=-0.38 upper=0 effort=1000.0 velocity=0.5; type fixed -> prismatic
- joint head_swivel: axis (none) -> 0 0 1; type fixed -> continuous
- joint left_gripper_joint: axis (none) -> 0 0 1; limit (none) -> lower=0.0 upper=0.548 effort=1000.0 velocity=0.5; type fixed -> revolute

Commit message: fix: add inertia

File: urdf/r2d2-example.urdf (robot description, URDF)
Before this commit: robot visual, 16 links, 15 joints
Links:
- link base_link: mass None -> 10; geometry collision cylinder length=0.6 radius=0.2; visual cylinder length=0.6 radius=0.2
